Commit message: Fix TOTG velocity=0, J4 sign convention, docs
- TimeParameterization: treat velocity=0 in URDF as unspecified (fallback
  1.0 rad/s).  Was causing ~100M s trajectories → Execute on Robot spinning.
- MyCobotBridge: add jointSignCorrection array [1,1,1,-1,1,1]; J4
  (joint5_to_joint4, index 3) is mechanically inverted vs URDF +Z convention.
  Correction applied in sendAngle, sendAngles, and pollAngles so physical arm
  and virtual arm stay in sync.  URDF axis left as 0 0 1 (standard).
- cobot.urdf: whitespace cleanup on joint5_to_joint4 axis attribute.
- APPROACH.md: add Section 9 Future Considerations.
- README.md: update status, testing steps, connect/disconnect notes.
- Add test_sign_convention.py and read_stream.py for hardware diagnostics.

File: Resources/cobot.urdf (robot description, URDF)
Before this commit: robot myCobot280, 8 links, 7 joints
Joints:
- joint joint5_to_joint4: axis  0 0 1 -> 0 0 1

Commit message: Fix J4 sign: URDF axis 0 0 -1, bridge all 1s; add Reload URDF button
The root cause of previous 'same behavior' reports: the app loads URDF from a
user-selected file path in memory — editing Resources/cobot.urdf on disk had no
effect until the file was re-picked in the Open dialog.  Fix:

- Resources/cobot.urdf: joint5_to_joint4 axis set to 0 0 -1, matching the
  physical hardware's positive rotation direction.  No bridge correction needed.
- MyCobotBridge.jointSignCorrection: reverted to [1,1,1,1,1,1] (all ones).
  Bridge corrections are reserved for joints where the hardware protocol sign
  differs from the URDF sign; J4 is now handled in the URDF itself.
- AppState.reloadURDF(): new method re-parses the last opened URL from disk,
  so on-disk URDF edits take effect instantly without re-selecting the file.
- ContentView: add 'Reload URDF' toolbar button (↺) next to 'Load URDF…';
  disabled when no file has been opened.

File: Resources/cobot.urdf (robot description, URDF)
Before this commit: robot myCobot280, 8 links, 7 joints
Joints:
- joint joint5_to_joint4: axis 0 0 1 -> 0 0 -1
